Commit message: Move docker package to simulator one

File: simulator/description/iris.xacro (robot description, xacro)
@@ -41,5 +41,5 @@
   </xacro:property>
   <!-- Included URDF Files -->
-  <xacro:include filename="$(find docker)/description/multirotor_base.xacro" />
+  <xacro:include filename="$(find simulator)/description/multirotor_base.xacro" />
   <!-- Instantiate multirotor_base_macro once -->
   <xacro:multirotor_base_macro

File: simulator/description/iris_base.xacro (robot description, xacro)
@@ -2,7 +2,7 @@
 <robot name="$(arg ns)" xmlns:xacro="http://ros.org/wiki/xacro">
   <xacro:property name="load" value="$(arg suspended_load)"/>
-  <xacro:include filename="$(find docker)/description/component_snippets.xacro" />
+  <xacro:include filename="$(find simulator)/description/component_snippets.xacro" />
   <!-- Instantiate iris "mechanics" -->
-  <xacro:include filename="$(find docker)/description/iris.xacro" />
+  <xacro:include filename="$(find simulator)/description/iris.xacro" />
   <!-- Instantiate a controller. -->
   <xacro:controller_plugin_macro

File: simulator/description/iris_base_load.xacro (robot description, xacro)
@@ -1,7 +1,8 @@
 <?xml version="1.0"?>
 <robot name="$(arg ns)" xmlns:xacro="http://ros.org/wiki/xacro">
-  <xacro:include filename="$(find docker)/description/component_snippets.xacro" />
+  <xacro:property name="load" value="true"/>
+  <xacro:include filename="$(find simulator)/description/component_snippets.xacro" />
   <!-- Instantiate iris "mechanics" -->
-  <xacro:include filename="$(find docker)/description/iris.xacro" />
+  <xacro:include filename="$(find simulator)/description/iris.xacro" />
   <!-- Instantiate a controller. -->
   <xacro:controller_plugin_macro
@@ -89,3 +90,35 @@
     </xacro:bag_plugin_macro>
   </xacro:if>
+  <xacro:if value="${load}">
+    <joint type="revolute" name="load_joint_1">
+      <parent link="base_link"/>
+      <origin rpy="0.0 0.0 0.0" xyz="0.0 0.0 0.7"/>
+      <child link="${namespace}/load"/>
+      <axis xyz="1 0 0"/>
+      <limit effort="50000" lower="-1.57079632679" upper="1.57079632679" velocity="10000"/>
+    </joint>
+    <!-- <link name="${namespace}/link_load"/>
+    <joint type="revolute" name="load_joint_2">
+      <parent link="${namespace}/link_load"/>
+      <origin rpy="0.0 0.0 0.0" xyz="0.0 0.0 0.7"/>
+      <child link="${namespace}/load"/>
+      <axis xyz="0 1 0"/>
+      <limit effort="50000" lower="-1.57079632679" upper="1.57079632679" velocity="10000"/>
+    </joint>
+ -->
+    <link name="${namespace}/load">
+      <inertial>
+        <inertia ixx="0.00001" ixy="0.0" ixz="0.0" iyy="0.00001" iyz="0.0" izz="0.00001"/>
+        <mass value="0.05"/>
+        <!-- [kg] -->
+        <origin rpy="0 0 0" xyz="0 0 0"/>
+      </inertial>
+      <origin rpy="0 0 0" xyz="0 0 0"/>
+      <visual name="visual">
+        <geometry>
+          <sphere radius="0.05"/>
+        </geometry>
+      </visual>
+    </link>
+  </xacro:if>
 </robot>

File: simulator/description/iris_base_multiple.xacro (robot description, xacro)
@@ -1,8 +1,7 @@
 <?xml version="1.0"?>
 <robot name="$(arg ns)" xmlns:xacro="http://ros.org/wiki/xacro">
-  <xacro:property name="load" value="true"/>
-  <xacro:include filename="$(find docker)/description/component_snippets.xacro" />
+  <xacro:include filename="$(find simulator)/description/component_snippets.xacro" />
   <!-- Instantiate iris "mechanics" -->
-  <xacro:include filename="$(find docker)/description/iris.xacro" />
+  <xacro:include filename="$(find simulator)/description/iris.xacro" />
   <!-- Instantiate a controller. -->
   <xacro:controller_plugin_macro
@@ -90,35 +89,3 @@
     </xacro:bag_plugin_macro>
   </xacro:if>
-  <xacro:if value="${load}">
-    <joint type="revolute" name="load_joint_1">
-      <parent link="base_link"/>
-      <origin rpy="0.0 0.0 0.0" xyz="0.0 0.0 0.7"/>
-      <child link="${namespace}/load"/>
-      <axis xyz="1 0 0"/>
-      <limit effort="50000" lower="-1.57079632679" upper="1.57079632679" velocity="10000"/>
-    </joint>
-    <!-- <link name="${namespace}/link_load"/>
-    <joint type="revolute" name="load_joint_2">
-      <parent link="${namespace}/link_load"/>
-      <origin rpy="0.0 0.0 0.0" xyz="0.0 0.0 0.7"/>
-      <child link="${namespace}/load"/>
-      <axis xyz="0 1 0"/>
-      <limit effort="50000" lower="-1.57079632679" upper="1.57079632679" velocity="10000"/>
-    </joint>
- -->
-    <link name="${namespace}/load">
-      <inertial>
-        <inertia ixx="0.00001" ixy="0.0" ixz="0.0" iyy="0.00001" iyz="0.0" izz="0.00001"/>
-        <mass value="0.05"/>
-        <!-- [kg] -->
-        <origin rpy="0 0 0" xyz="0 0 0"/>
-      </inertial>
-      <origin rpy="0 0 0" xyz="0 0 0"/>
-      <visual name="visual">
-        <geometry>
-          <sphere radius="0.05"/>
-        </geometry>
-      </visual>
-    </link>
-  </xacro:if>
 </robot>
